Commit message: update

File: urdf2model/models/HYUMM/hyumm.urdf (robot description, URDF)
Before this commit: robot hyumm, 16 links, 15 joints
Links:
- removed link wheel_left_back
- removed link wheel_left_front
- removed link wheel_right_back
- removed link wheel_right_front
- link base_link: mass 50.03647319 -> 53.53736408
Joints:
- removed joint joint_left_back
- removed joint joint_left_front
- removed joint joint_right_back
- removed joint joint_right_front

File: urdf2model/models/HYUMM/mobile.urdf (robot description, URDF)
Before this commit: robot hyumob, 4 links, 3 joints
Links:
- link base_link: mass 53.53736408 -> 50.0; geometry collision mesh filename=meshes/stl/base.STL; visual mesh filename=meshes/stl/base.STL

File: urdf2model/models/indy7/indy7.urdf (robot description, URDF)
Before this commit: robot indy7, 8 links, 7 joints
Links:
- link link0: geometry visual mesh filename=meshes/stl/Indy7_0.stl
- link link1: geometry visual mesh filename=meshes/stl/Indy7_1.stl
- link link2: geometry visual mesh filename=meshes/stl/Indy7_2.stl
- link link3: geometry visual mesh filename=meshes/stl/Indy7_3.stl
- link link4: geometry visual mesh filename=meshes/stl/Indy7_4.stl
- link link5: geometry visual mesh filename=meshes/stl/Indy7_5.stl
- link link6: geometry visual mesh filename=meshes/stl/Indy7_6.stl

Commit message: update

File: urdf2model/models/HYUMM/hyumm.urdf (robot description, URDF)
Before this commit: robot hyumm, 12 links, 11 joints
Links:
- link lin_x_link: mass 0.000001 -> 0
- link lin_y_link: mass 0.000001 -> 0
- link tcp: mass 0.000001 -> 0
- link world: mass 0.000001 -> 0

File: urdf2model/models/HYUMM/hyumob.urdf (robot description, URDF)
Before this commit: robot hyumob, 4 links, 3 joints
Links:
- link lin_x_link: mass 0.000001 -> 0
- link lin_y_link: mass 0.000001 -> 0
- link world: mass 0.000001 -> 0
