Commit message: KARM_EM

File: urdf2model/models/HYUMM/hyumob_floating.urdf (robot description, URDF)
Before this commit: robot hyumob_floating, 2 links, 1 joints
Links:
- added link link0, mass 1.67030785; visual mesh filename=meshes/stl/Indy7_0.stl
Joints:
- added joint base_flange: type fixed, parent base_link, child link0, origin xyz=0.3 0 0.228 rpy=0 0 0

File: urdf2model/models/caesar/KARM_EM.urdf (robot description, URDF)
Before this commit: robot KARM_EM, 10 links, 9 joints
Links:
- removed link ASM_HOUSING_T_EM
- removed link ASM_J1_EM
- removed link ASM_J2_EM
- removed link ASM_J3_EM
- removed link ASM_J4_EM
- removed link ASM_J5_EM
- removed link ASM_J6_EM
- removed link ASM_J7_EM
- added link ASM_LINK_0_EM, mass 0.47278619  ; collision mesh filename=../meshes/ASM_LINK_0_EM.STL; visual mesh filename=../meshes/ASM_LINK_0_EM.STL
- added link ASM_LINK_1_EM, mass 8.41295125; collision mesh filename=../meshes/ASM_LINK_1_EM.STL; visual mesh filename=../meshes/ASM_LINK_1_EM.STL
- added link ASM_LINK_2_EM, mass 1.08543372  ; collision mesh filename=../meshes/ASM_LINK_2_EM.STL; visual mesh filename=../meshes/ASM_LINK_2_EM.STL
- added link ASM_LINK_3_EM, mass 10.45122582; collision mesh filename=../meshes/ASM_LINK_3_EM.STL; visual mesh filename=../meshes/ASM_LINK_3_EM.STL
- added link ASM_LINK_4_EM, mass 1.08543372; collision mesh filename=../meshes/ASM_LINK_4_EM.STL; visual mesh filename=../meshes/ASM_LINK_4_EM.STL
- added link ASM_LINK_5_EM, mass 8.50980173 ; collision mesh filename=../meshes/ASM_LINK_5_EM.STL; visual mesh filename=../meshes/ASM_LINK_5_EM.STL
- added link ASM_LINK_6_EM, mass 5.47249246; collision mesh filename=../meshes/ASM_LINK_6_EM.STL; visual mesh filename=../meshes/ASM_LINK_6_EM.STL
- added link ASM_LINK_7_EM, mass 0.47459064 ; collision mesh filename=../meshes/ASM_LINK_7_EM.STL; visual mesh filename=../meshes/ASM_LINK_7_EM.STL
Joints:
- joint eef_fixed: parent ASM_J7_EM -> ASM_LINK_7_EM
- joint joint1: child ASM_HOUSING_T_EM -> ASM_LINK_1_EM; origin xyz=0 0 0.128 rpy=0 0 0 -> xyz=0 0 0.094 rpy=0 0 0; parent ASM_J1_EM -> ASM_LINK_0_EM
- joint joint2: child ASM_J2_EM -> ASM_LINK_2_EM; origin xyz=0 0.0915 0.128 rpy=0 0 0 -> xyz=0 -0.104 0.105 rpy=0 0 0; parent ASM_HOUSING_T_EM -> ASM_LINK_1_EM
- joint joint3: child ASM_J3_EM -> ASM_LINK_3_EM; origin xyz=0 0.0915 0.4695 rpy=0 0.0 0 -> xyz=0 -0.088 0.129 rpy=0 0.0 0; parent ASM_J2_EM -> ASM_LINK_2_EM
- joint joint4: child ASM_J4_EM -> ASM_LINK_4_EM; origin xyz=0.0 -0.0915 0.3955 rpy=0 0 0 -> xyz=0 0.104 0.798 rpy=0 0 0; parent ASM_J3_EM -> ASM_LINK_3_EM
- joint joint5: child ASM_J5_EM -> ASM_LINK_5_EM; origin xyz=0 -0.0915 0.1395 rpy=0 0 0 -> xyz=0 0.088 0.129 rpy=0 0 0; parent ASM_J4_EM -> ASM_LINK_4_EM
- joint joint6: child ASM_J6_EM -> ASM_LINK_6_EM; origin xyz=0 -0.0915 0.3955 rpy=0 0 0 -> xyz=0 0.104 0.406 rpy=0 0 0; parent ASM_J5_EM -> ASM_LINK_5_EM
- joint joint7: child ASM_J7_EM -> ASM_LINK_7_EM; origin xyz=0 -0.0915 0.128 rpy=0 0 0 -> xyz=0 0.088 0.121 rpy=0 0 0; parent ASM_J6_EM -> ASM_LINK_6_EM
- joint world_fixed: child ASM_J1_EM -> ASM_LINK_0_EM
