Commit message: update

File: urdf2model/models/caesar/ASM_KARI_ARM_URDF.urdf (robot description, URDF)
Before this commit: robot ASM_KARI_ARM_URDF, 10 links, 9 joints
Links:
- link base: geometry collision mesh filename=meshes/ASM_J0.STL; visual mesh filename=meshes/ASM_J0.STL
- link link1: geometry collision mesh filename=meshes/ASM_J1.STL; visual mesh filename=meshes/ASM_J1.STL
- link link2: geometry collision mesh filename=meshes/ASM_J2.STL; visual mesh filename=meshes/ASM_J2.STL
- link link3: geometry collision mesh filename=meshes/ASM_J3.STL; visual mesh filename=meshes/ASM_J3.STL
- link link4: geometry collision mesh filename=meshes/ASM_J4.STL; visual mesh filename=meshes/ASM_J4.STL
- link link5: geometry collision mesh filename=meshes/ASM_J5.STL; visual mesh filename=meshes/ASM_J5.STL
- link link6: geometry collision mesh filename=meshes/ASM_J6.STL; visual mesh filename=meshes/ASM_J6.STL
- link link7: geometry collision mesh filename=meshes/ASM_J7.STL; visual mesh filename=meshes/ASM_J7.STL
Joints:
- joint joint4: origin xyz=0.0 0.08800000 0.80000000 rpy=0 0 0 -> xyz=0.0 -0.088 0.8 rpy=0 0 0
- joint joint5: origin xyz=0.0 0.10400000 0.13100000 rpy=0 0 0 -> xyz=0.0 -0.10400000 0.13100000 rpy=0 0 0
- joint joint6: origin xyz=0.0 0.07100000 0.40800000  rpy=0 0 0 -> xyz=0.0 -0.07100000 0.40800000  rpy=0 0 0
- joint joint7: origin xyz=0.0 0.12100000 0.08800000 rpy=0 0 0 -> xyz=0.0 -0.12100000 0.08800000 rpy=0 0 0
