Commit message: update

File: urdf2model/models/caesar/KARM_EM.urdf (robot description, URDF)
Before this commit: robot KARM_EM, 10 links, 9 joints
Links:
- link ASM_LINK_0_EM: mass 0.47278619   -> 0.47278619
- link ASM_LINK_2_EM: mass 1.08543372   -> 1.08543372
- link ASM_LINK_5_EM: mass 8.50980173  -> 8.50980173
- link ASM_LINK_7_EM: mass 0.47459064  -> 0.47459064

File: urdf2model/models/indy7/indy7.urdf (robot description, URDF)
Before this commit: robot indy7, 8 links, 7 joints
Joints:
- joint indy7_tcp: origin xyz=0 0 0.23 rpy=0 0 0 -> xyz=0 0 0.0795 rpy=0 0 0

File: urdf2model/models/indy7/indy7_dualarm.urdf (robot description, URDF)
Before this commit: robot indy7_dualarm, 9 links, 8 joints
Links:
- removed link link0
- removed link link1
- removed link link2
- removed link link3
- removed link link4
- removed link link5
- removed link link6
- removed link tcp
- added link link0_l, mass 1.67030785; visual mesh filename=meshes/stl/Indy7_0.stl
- added link link1_l, mass 11.44444535; visual mesh filename=meshes/stl/Indy7_1.stl
- added link link2_l, mass 5.84766553; visual mesh filename=meshes/stl/Indy7_2.stl
- added link link3_l, mass 2.68206064; visual mesh filename=meshes/stl/Indy7_3.stl
- added link link4_l, mass 2.12987371; visual mesh filename=meshes/stl/Indy7_4.stl
- added link link5_l, mass 2.22412271; visual mesh filename=meshes/stl/Indy7_5.stl
- added link link6_l, mass 0.38254932; visual mesh filename=meshes/stl/Indy7_6.stl
- added link tcp_l, mass 0.000001
Joints:
- removed joint indy7_tcp
- removed joint joint0
- removed joint joint1
- removed joint joint2
- removed joint joint3
- removed joint joint4
- removed joint joint5
- removed joint world_joint
- added joint indy7_tcp_l: type fixed, parent link6_l, child tcp_l, origin xyz=0 0 0.06 rpy=0 0 0
- added joint joint0_l: type revolute, parent link0_l, child link1_l, origin xyz=0 0 0.0775 rpy=0 0 0, axis 0 0 1, limit lower=-3.0543261909900763 upper=3.0543261909900763 effort=10 velocity=1
- added joint joint1_l: type revolute, parent link1_l, child link2_l, origin xyz=0 -0.10900000 0.22200000 rpy=1.5707963267948966 1.5707963267948966 0, axis 0 0 1, limit lower=-3.0543261909900763 upper=3.0543261909900763 effort=10 velocity=1
- added joint joint2_l: type revolute, parent link2_l, child link3_l, origin xyz=-0.45000000 +0.00000000 -0.03050000 rpy=0 0 0, axis 0 0 1, limit lower=-3.0543261909900763 upper=3.0543261909900763 effort=10 velocity=1
- added joint joint3_l: type revolute, parent link3_l, child link4_l, origin xyz=-0.26700000 +0.00000000 -0.07500000 rpy=-1.5707963267948966 0 1.5707963267948966, axis 0 0 1, limit lower=-3.0543261909900763 upper=3.0543261909900763 effort=10 velocity=1
- added joint joint4_l: type revolute, parent link4_l, child link5_l, origin xyz=+0.00000000 -0.11400000 +0.08300000 rpy=1.5707963267948966 1.5707963267948966 0, axis 0 0 1, limit lower=-3.0543261909900763 upper=3.0543261909900763 effort=10 velocity=1
- added joint joint5_l: type revolute, parent link5_l, child link6_l, origin xyz=-0.16800000 +0.00000000 +0.06900000 rpy=-1.5707963267948966 0 1.5707963267948966, axis 0 0 1, limit lower=-3.752457891787808 upper=3.752457891787808 effort=10 velocity=1
- added joint world_joint_l: type fixed, parent world, child link0_l, origin xyz=0 0.1551 1.2924 rpy=2.094407804564866 0 3.141592
