Commit message: update

File: urdf2model/models/NRMK/indyrp2/indyrp2.urdf (robot description, URDF)
Before this commit: robot indyrp2, 9 links, 8 joints
Links:
- link link0: geometry visual mesh filename=meshes/stl/indyrp2/IndyRP2_0.stl
- link link1: geometry visual mesh filename=meshes/stl/indyrp2/IndyRP2_1.stl
- link link2: geometry visual mesh filename=meshes/stl/indyrp2/IndyRP2_2.stl
- link link3: geometry visual mesh filename=meshes/stl/indyrp2/IndyRP2_3.stl
- link link4: geometry visual mesh filename=meshes/stl/indyrp2/IndyRP2_4.stl
- link link5: geometry visual mesh filename=meshes/stl/indyrp2/IndyRP2_5.stl
- link link6: geometry visual mesh filename=meshes/stl/indyrp2/IndyRP2_6.stl
- link link7: geometry visual mesh filename=meshes/stl/indyrp2/IndyRP2_7.stl
