Commit message: update

File: urdf2model/models/HDRobotics/yl012/yl012_sat.urdf (robot description, URDF)
Before this commit: robot yl102_sat, 11 links, 10 joints
Joints:
- removed joint sat_fixed
- added joint flange_fixed: type fixed, parent link6, child link_sat, origin xyz=0 0 0.07385 rpy=0 0 0, axis 0 0 0

File: urdf2model/models/HDRobotics/yl012/yl012_sat_core.urdf (robot description, URDF)
Before this commit: robot yl102_sat_core, 11 links, 10 joints
Links:
- added link link_flange, mass 0.71; collision mesh filename=meshes/link_FT.stl; visual mesh filename=meshes/link_FT.stl
- added link link_tcp_CoM, mass 00
- link link_ft: mass 0.71 -> 00; geometry 
Joints:
- added joint flange_fixed: type fixed, parent link6, child link_flange, origin xyz=0 0 0.07385 rpy=0 0 0, axis 0 0 0
- added joint tcp_CoM_fixed: type fixed, parent link_sat, child link_tcp_CoM, origin xyz=-0.00001166 -0.00000932 -0.04673098 rpy=0 0 0, axis 0 0 0
- joint core_fixed: origin xyz=0 0 0.0412 rpy=0 0 0 -> xyz=0 0 0.01 rpy=0 0 0
- joint ft_fixed: origin xyz=0 0 0.07385 rpy=0 0 0 -> xyz=0 0 0.0312 rpy=0 0 0; parent link6 -> link_flange
