Commit message: update

File: urdf2model/models/HDRobotics/yl012/yl012_sat_core.urdf (robot description, URDF)
Before this commit: robot yl102_sat_core, 13 links, 12 joints
Joints:
- joint core_fixed: origin xyz=0 0 0.01 rpy=0 0 0 -> xyz=0.00001166 0.00000932 -0.12976902 rpy=0 0 0; parent link_ft -> link_tcp_CoM
- joint tcp_CoM_fixed: origin xyz=-0.00001166 -0.00000932 -0.04673098 rpy=0 0 0 -> xyz=-0.00001166 -0.00000932 0.13976902 rpy=0 0 0; parent link_sat -> link_ft
