Commit message: update

File: urdf2model/models/hyu_spa/hyu_spa.urdf (robot description, URDF)
Before this commit: robot space_arm_base, 10 links, 9 joints
Links:
- removed link link7
- removed link world
- link link0: mass 1.6 -> 14.299; geometry visual mesh filename=meshes/stl/hyu_spa_0.stl
- link link1: mass 0.83842732 -> 0.63842732; geometry visual mesh filename=meshes/stl/hyu_spa_1.stl
- link link2: mass 0.70158865 -> 0.60158865; geometry visual mesh filename=meshes/stl/hyu_spa_2.stl
- link link3: geometry visual mesh filename=meshes/stl/hyu_spa_3.stl
- link link4: geometry visual mesh filename=meshes/stl/hyu_spa_4.stl
- link link5: geometry visual mesh filename=meshes/stl/hyu_spa_5.stl
- link link6: geometry visual mesh filename=meshes/stl/hyu_spa_6.stl
Joints:
- removed joint joint6
- removed joint joint7
- removed joint joint_tcp
- removed joint world_fixed
- added joint joint0: type revolute, parent link0, child link1, origin xyz=0 -0.3107 1.567 rpy=0 0 0, axis 0 1 0, limit lower=-3.0543261909900763 upper=3.0543261909900763 effort=10 velocity=1
- added joint tcp_fixed: type fixed, parent link6, child tcp, origin xyz=0 0 0.0795 rpy=0 0 0
- joint joint1: axis 0 0 1 -> 1 0 0; child link1 -> link2; origin xyz=0 0 -0.2287 rpy=0 0 0 -> xyz=0 -0.054 0 rpy=0 0 0; parent link0 -> link1
- joint joint2: axis 1 0 0 -> 0 0 1; child link2 -> link3; origin xyz=0 0 -0.054 rpy=0 0 0 -> xyz=0 0 -0.1458 rpy=0 0 0; parent link1 -> link2
- joint joint3: axis 0 0 1 -> 0 1 0; child link3 -> link4; origin xyz=0 0 -0.1458 rpy=0 0 0 -> xyz=0 0 -0.1542 rpy=0 0 0; parent link2 -> link3
- joint joint4: axis 1 0 0 -> 0 0 1; child link4 -> link5; origin xyz=0 0 -0.1542 rpy=0 0 0 -> xyz=0 0 -0.1458 rpy=0 0 0; parent link3 -> link4
- joint joint5: axis 0 0 1 -> 1 0 0; child link5 -> link6; limit lower=-3.0543261909900763 upper=3.0543261909900763 effort=10 velocity=1 -> lower=-3.752457891787808 upper=3.752457891787808 effort=10 velocity=1; origin xyz=0 0 -0.1458 rpy=0 0 0 -> xyz=0 0 -0.1542 rpy=0 0 0; parent link4 -> link5

File: urdf2model/models/space_arm/space_arm_tip.urdf (robot description, URDF)
Before this commit: robot space_arm_tip, 10 links, 9 joints
Links:
- link link1: mass 0.63842732 -> 0.59063954
- link link2: mass 0.60158865 -> 0.74955005
- link link3: mass 0.74955005 -> 0.57916453
- link link4: mass 0.57916453 -> 0.74955005
- link link5: mass 0.74955005 -> 0.70158865
- link link6: mass 0.59063954 -> 0.83842732
- link link7: mass 1.4 -> 1.6

File: urdf2model/models/space_arm/space_arm_virtual.urdf (robot description, URDF)
Before this commit: robot space_arm_base, 10 links, 9 joints
Links:
- added link VirtualLink_p1, mass 0.0000001; collision box size=0.00 0.00 0.00
- added link VirtualLink_p2, mass 0.0000001; collision box size=0.00 0.00 0.00
- added link VirtualLink_p3, mass 0.0000001; collision box size=0.00 0.00 0.00
- added link VirtualLink_r1, mass 0.0000001; collision box size=0.00 0.00 0.00
- added link VirtualLink_r2, mass 0.0000001; collision box size=0.00 0.00 0.00
- link link0: mass 1.6 -> 1.4
- link link1: mass 0.83842732 -> 0.63842732
- link link2: mass 0.70158865 -> 0.60158865
Joints:
- removed joint joint7
- removed joint joint_tcp
- removed joint world_fixed
- added joint VirtualJoint_px: type prismatic, parent world, child VirtualLink_p1, origin xyz=0 0 0 rpy=0 0 0, axis 1 0 0, limit lower=-1000 upper=1000 effort=100 velocity=1000
- added joint VirtualJoint_py: type prismatic, parent VirtualLink_p1, child VirtualLink_p2, origin xyz=0 0 0 rpy=0 0 0, axis 0 1 0, limit lower=-1000 upper=1000 effort=100 velocity=1000
- added joint VirtualJoint_pz: type prismatic, parent VirtualLink_p2, child VirtualLink_p3, origin xyz=0 0 0 rpy=0 0 0, axis 0 0 1, limit lower=-1000 upper=1000 effort=100 velocity=1000
- added joint VirtualJoint_rx: type revolute, parent VirtualLink_p3, child VirtualLink_r1, origin xyz=0 0 0 rpy=0 0 0, axis 1 0 0, limit lower=-1000 upper=1000 effort=100 velocity=1000
- added joint VirtualJoint_ry: type revolute, parent VirtualLink_r1, child VirtualLink_r2, origin xyz=0 0 0 rpy=0 0 0, axis 0 1 0, limit lower=-1000 upper=1000 effort=100 velocity=1000
- added joint VirtualJoint_rz: type revolute, parent VirtualLink_r2, child link0, origin xyz=0 0 0 rpy=0 0 0, axis 0 0 1, limit lower=-1000 upper=1000 effort=100 velocity=1000
- added joint joint0: type revolute, parent link0, child link1, origin xyz=0 0 -0.2287 rpy=0 0 0, axis 0 0 1, limit lower=-3.0543261909900763 upper=3.0543261909900763 effort=10 velocity=1
- added joint tcp_fixed: type fixed, parent link7, child tcp, origin xyz=0 0 -0.2357 rpy=0 0 0
- joint joint1: axis 0 0 1 -> 1 0 0; child link1 -> link2; origin xyz=0 0 -0.2287 rpy=0 0 0 -> xyz=0 0 -0.054 rpy=0 0 0; parent link0 -> link1
- joint joint2: axis 1 0 0 -> 0 0 1; child link2 -> link3; origin xyz=0 0 -0.054 rpy=0 0 0 -> xyz=0 0 -0.1458 rpy=0 0 0; parent link1 -> link2
- joint joint3: axis 0 0 1 -> 1 0 0; child link3 -> link4; origin xyz=0 0 -0.1458 rpy=0 0 0 -> xyz=0 0 -0.1542 rpy=0 0 0; parent link2 -> link3
- joint joint4: axis 1 0 0 -> 0 0 1; child link4 -> link5; origin xyz=0 0 -0.1542 rpy=0 0 0 -> xyz=0 0 -0.1458 rpy=0 0 0; parent link3 -> link4
- joint joint5: axis 0 0 1 -> 1 0 0; child link5 -> link6; limit lower=-3.0543261909900763 upper=3.0543261909900763 effort=10 velocity=1 -> lower=-3.752457891787808 upper=3.752457891787808 effort=10 velocity=1; origin xyz=0 0 -0.1458 rpy=0 0 0 -> xyz=0 0 -0.1542 rpy=0 0 0; parent link4 -> link5
- joint joint6: axis 1 0 0 -> 0 0 1; child link6 -> link7; origin xyz=0 0 -0.1542 rpy=0 0 0 -> xyz=0 0 -0.054 rpy=0 0 0; parent link5 -> link6
