Commit message: update: indy12_v2

File: urdf2model/models/NRMK/indy12_v2/indy12_v2.urdf (robot description, URDF)
Before this commit: robot indy12_v2, 9 links, 8 joints
Links:
- added link RFT64-6A01, mass 0.175
- added link tool_changer, mass 2.125
- added link tool_plange, mass 0.300
- link link0: geometry visual mesh filename=meshes/indy12_v2/link0.stl
- link link1: geometry visual mesh filename=meshes/indy12_v2/link1.stl
- link link2: geometry visual mesh filename=meshes/indy12_v2/link2.stl
- link link3: mass 8.45645221 -> 5.0597333; geometry visual mesh filename=meshes/indy12_v2/link3.stl
- link link4: geometry visual mesh filename=meshes/indy12_v2/link4.stl
- link link5: geometry visual mesh filename=meshes/indy12_v2/link5.stl
- link link6: geometry visual mesh filename=meshes/indy12_v2/link6.stl
- link link7: geometry visual mesh filename=meshes/indy12_v2/link7.stl
Joints:
- added joint RFT_fixed: type fixed, parent tool_plange, child RFT64-6A01, origin xyz=0 0 0.0641 rpy=0 0 0
- added joint changer_fixed: type fixed, parent RFT64-6A01, child tool_changer, origin xyz=0 0 0.03 rpy=0 0 0
- added joint plange_fixed: type fixed, parent link7, child tool_plange, origin xyz=0 0 0.0841 rpy=0 0 0
- joint tcp_fixed: parent link7 -> tool_changer

Commit message: update: indy12_v2

File: urdf2model/models/NRMK/indy12_v2/indy12_v2.urdf (robot description, URDF)
Before this commit: robot indy12_v2, 12 links, 11 joints
Links:
- link link0: geometry visual mesh filename=meshes/stl/indy12_v2/link0.stl
- link link1: geometry visual mesh filename=meshes/stl/indy12_v2/link1.stl
- link link2: geometry visual mesh filename=meshes/stl/indy12_v2/link2.stl
- link link3: mass 5.0597333 -> 8.45645221; geometry visual mesh filename=meshes/stl/indy12_v2/link3.stl
- link link4: geometry visual mesh filename=meshes/stl/indy12_v2/link4.stl
- link link5: geometry visual mesh filename=meshes/stl/indy12_v2/link5.stl
- link link6: geometry visual mesh filename=meshes/stl/indy12_v2/link6.stl
- link link7: geometry visual mesh filename=meshes/stl/indy12_v2/link7.stl

Commit message: update:

File: urdf2model/models/NRMK/indy12_v2/indy12_v2.urdf (robot description, URDF)
Before this commit: robot indy12_v2, 12 links, 11 joints
Links:
- link link0: geometry visual mesh filename=meshes/indy12_v2/link0.stl
- link link1: geometry visual mesh filename=meshes/indy12_v2/link1.stl
- link link2: geometry visual mesh filename=meshes/indy12_v2/link2.stl
- link link3: geometry visual mesh filename=meshes/indy12_v2/link3.stl
- link link4: geometry visual mesh filename=meshes/indy12_v2/link4.stl
- link link5: geometry visual mesh filename=meshes/indy12_v2/link5.stl
- link link6: geometry visual mesh filename=meshes/indy12_v2/link6.stl
- link link7: geometry visual mesh filename=meshes/indy12_v2/link7.stl
Joints:
- joint joint5: origin xyz=0 -0.12900000 0.36250000 rpy=0 0 0 -> xyz=0 0.12900000 0.36250000 rpy=0 0 0
- joint joint6: origin xyz=0 -0.07950000 +0.07455 rpy=0 0 0 -> xyz=0 0.07950000 +0.07455 rpy=0 0 0
