Commit message: update: KR120,250, indy12_v2_sat

File: urdf2model/models/KUKA/kuka_kr120/kuka_kr_120_sat.urdf (robot description, URDF)
Before this commit: robot kuka_kr_120_sat, 16 links, 15 joints
Links:
- link FTSensor: mass 0.001 -> 0.0
- link TGT: mass 0.001 -> 500.0
- link TGT_fixture: mass 0.001 -> 0.0
- link TGT_launcherring: mass 0.001 -> 0.0
- link TGT_pannel: mass 0.001 -> 0.0

File: urdf2model/models/NRMK/indy12_v2/indy12_v2_sat.urdf (robot description, URDF)
Before this commit: robot indy12_v2_sat, 20 links, 19 joints
Links:
- added link FTSensor, mass 0.000
- added link l_tcp, mass 0
Joints:
- added joint CRS_fixed: type fixed, parent FTSensor, child l_CRS_black, origin xyz=0.0 0.0 0.0 rpy=0.0 0  0
- added joint ft_sensor_joint: type fixed, parent l_tcp, child FTSensor, origin xyz=0.0 0.0 0.1048 rpy=0.0 0  3.1415926536
- joint Px: limit lower=-2 upper=2 effort=10000 velocity=1000 -> lower=-20 upper=20 effort=10000 velocity=1000
- joint Py: limit lower=-1 upper=1 effort=10000 velocity=1000 -> lower=-10 upper=10 effort=10000 velocity=1000
- joint Rx: child l_CRS_black -> l_tcp
- joint sat_to_indy12_fixed: parent l_CRS_black -> FTSensor

Commit message: feat: kuka update

File: urdf2model/models/KUKA/kuka_kr120/kuka_kr_120_sat.urdf (robot description, URDF)
Before this commit: robot kuka_kr_120_sat, 16 links, 15 joints
Links:
- removed link FTSensor
- removed link TGT
- removed link TGT_fixture
- removed link TGT_launcherring
- removed link TGT_pannel
- removed link base_link
- removed link link1
- removed link link2
- removed link link3
- removed link link4
- removed link link5
- removed link link6
- removed link plate_link
- removed link tcp
- added link r_FTSensor, mass 0.001; visual mesh filename=meshes/kuka_120_ft_sensor.stl
- added link r_TGT, mass 0.001; visual mesh filename=meshes/TGT.stl
- added link r_TGT_fixture, mass 0.001; visual mesh filename=meshes/TGT_fixture.stl
- added link r_TGT_launcherring, mass 0.001; visual mesh filename=meshes/TGT_launcherring.stl
- added link r_TGT_pannel, mass 0.001; visual mesh filename=meshes/TGT_pannel.stl
- added link r_base_link, mass 257.693; visual mesh filename=meshes/kuka_kr_120_base_link.stl
- added link r_link1, mass 254.573; visual mesh filename=meshes/kuka_kr_120_link1.stl
- added link r_link2, mass 331.528; visual mesh filename=meshes/kuka_kr_120_link2.stl
- added link r_link3, mass 172.325; collision mesh filename=meshes/kuka_kr_120_link3.stl; visual mesh filename=meshes/kuka_kr_120_link3.stl
- added link r_link4, mass 18.8575; visual mesh filename=meshes/kuka_kr_120_link4.stl
- added link r_link5, mass 37.375; visual mesh filename=meshes/kuka_kr_120_link5.stl
- added link r_link6, mass 3.13638; visual mesh filename=meshes/kuka_kr_120_link6.stl
- added link r_plate_link; visual mesh filename=meshes/right_plate.stl
- added link r_tcp, mass 0
Joints:
- removed joint TGT_fixed
- removed joint TGT_fixture_fixed
- removed joint TGT_launchering_fixed
- removed joint TGT_pannel_fixed
- removed joint ft_sensor_joint
- removed joint joint1
- removed joint joint2
- removed joint joint3
- removed joint joint4
- removed joint joint5
- removed joint joint6
- removed joint plate_base_joint
- removed joint tcp_joint
- removed joint world_joint
- added joint r_TGT_fixed: type fixed, parent r_FTSensor, child r_TGT, origin xyz=0.0 0.0 0.0 rpy=0.0 0.0 0.0
- added joint r_TGT_fixture_fixed: type fixed, parent r_FTSensor, child r_TGT_fixture, origin xyz=0.0 0.0 0.0 rpy=0.0 0.0 0.0
- added joint r_TGT_launchering_fixed: type fixed, parent r_FTSensor, child r_TGT_launcherring, origin xyz=0.0 0.0 0.0 rpy=0.0 0.0 0.0
- added joint r_TGT_pannel_fixed: type fixed, parent r_FTSensor, child r_TGT_pannel, origin xyz=0.0 0.0 0.0 rpy=0.0 0.0 0.0
- added joint r_ft_sensor_joint: type fixed, parent r_tcp, child r_FTSensor, origin xyz=0.0 0.0 0.08588 rpy=0.0 0  3.1415926536
- added joint r_joint1: type revolute, parent r_base_link, child r_link1, origin xyz=0.0 0.0 0.2356 rpy=3.14159265358 0.0 0.0, axis 0 0 1, limit lower=-3.2289 upper=3.2289 effort=100000 velocity=1000
- added joint r_joint2: type revolute, parent r_link1, child r_link2, origin xyz=0.33 0.0 -0.4094 rpy=1.57079632679 0.0 0.0, axis 0 0 1, limit lower=-2.4435 upper=-0.0873 effort=100000 velocity=1000
- added joint r_joint3: type revolute, parent r_link2, child r_link3, origin xyz=1.15 0.0 -0.095 rpy=0.0 0.0 0.0, axis 0 0 1, limit lower=-2.0944 upper=2.9322 effort=100000 velocity=1000
- added joint r_joint4: type revolute, parent r_link3, child r_link4, origin xyz=0.8785 -0.115 0.095 rpy=0.0 -1.57079632679 0.0, axis 0 0 1, limit lower=-6.1087 upper=6.1087 effort=100000 velocity=1000
- added joint r_joint5: type revolute, parent r_link4, child r_link5, origin xyz=0.059 0.0 -0.3415 rpy=0.0 1.57079632679 0.0, axis 0 0 1, limit lower=-2.1817 upper=2.1817 effort=100000 velocity=1000
- added joint r_joint6: type revolute, parent r_link5, child r_link6, origin xyz=0.195 0.0 -0.059 rpy=0.0 -1.57079632679 0.0, axis 0 0 1, limit lower=-6.1087 upper=6.1087 effort=100000 velocity=1000
- added joint r_plate_base_joint: type fixed, parent r_plate_link, child r_base_link, origin xyz=0.0 0.0 0.05 rpy=0.0 0.0 3.14159265358
- added joint r_tcp_joint: type fixed, parent r_link6, child r_tcp, origin xyz=0.0 0.0 -0.02 rpy=3.1415926536 0.0 1.5707963268
- added joint r_world_joint: type fixed, parent world, child r_plate_link, origin xyz=0 0 0 rpy=0.0 0.0 3.141592
- joint tcp_CoM_fixed: parent TGT -> r_TGT

Commit message: fix: kuka kr120

File: urdf2model/models/KUKA/kuka_kr120/kuka_kr_120_sat.urdf (robot description, URDF)
Before this commit: robot kr_120_plate_kr_250_rail, 16 links, 15 joints
Joints:
- joint tcp_CoM_fixed: origin xyz=-0.00001166 -0.00000932 -0.04673098 rpy=0 0 0 -> xyz=-0.0290 0.0076 0.0677 rpy=0 0 0
