Commit message: karm_em_v2_sat

File: urdf2model/models/KUKA/kuka_kr120/kuka_kr_120_sat.urdf (robot description, URDF)
Before this commit: robot kuka_kr_120_sat, 16 links, 15 joints
Joints:
- joint r_ft_sensor_joint: origin xyz=0.0 0.0 0.08588 rpy=0.0 0  3.1415926536 -> xyz=0.0 0.0 0.08588 rpy=0 0 0
